File: kicad/fiberPCB/test01.kicad_pcb (KiCad board)
At the start: 2 copper layers, 33 x 24 mm, 23 parts, among them J1 Conn_01x01_Male, J2 Conn_01x01_Male, J3 Conn_01x01_Male, J4 Conn_01x01_Male, J5 Conn_01x01_Male, J6 Conn_01x01_Male, J7 Conn_01x01_Male, J8 Conn_01x01_Male, P5 Conn_01x10_Male

Commit message: made test01 pattern
Parts:
- J1, J2, J3, J4, J5, J6, J7, J8: footprint Pin_Headers:Pin_Header_Straight_1x01_Pitch2.54mm -> fiberPCB:Checkpoint
- moved J1 4.74 mm to (146.8, 36.6)
- moved J5 4.74 mm to (146.8, 39.1)
- moved J6 3.66 mm to (148.1, 40.4)
- moved J2 3.66 mm to (148.1, 37.8)
- moved J3 2.88 mm to (149.4, 39.1)
- moved J7 2.88 mm to (149.4, 41.7)
- moved J4 2.69 mm to (150.6, 40.4)
- moved J8 1.99 mm to (150.6, 42.9)
- moved R0603(0201) 0.27 mm to (155.8, 52.8)
Routing:
- net Net-(J1-Pad1): track 93.3 -> 89.9 mm
- net Net-(J4-Pad1): track 79.6 -> 81.4 mm
- net Net-(J2-Pad1): track 88.8 -> 87.4 mm
- net Net-(J3-Pad1): track 85.4 -> 84.8 mm
Other:
- board size 33 x 24 mm -> 31 x 22.5 mm
- rule trace_min: 0.2 -> 0.0254
- rule via_min_size: 0.4 -> 0.0254
- board text added: "10/20mil"
- board text added: "2.5/5"
- board text added: "22.5x31mm"
- board text added: "M3"
- board text added: "by Shingo"
- board text added: "fiberPCB"
- board text added: "test01"
- board text removed: "15/20mil"
- board text removed: "24x33mm"
- board text removed: "9.84/10"
- board text removed: "S.Hisakawa"

Commit message: rewire test01 pattern
Parts:
- moved PH_Pitch1.00 14.6 mm to (165.4, 47.8), turned to 0 degrees
- moved PH_Pitch1.27 11.4 mm to (165.4, 45.9), turned to 0 degrees
- moved PH_Pitch2.00 8.58 mm to (165.8, 43.8), turned to 0 degrees
- moved P.1 7.81 mm to (159.8, 41.9)
- moved J1 7.72 mm to (153.7, 40.0)
- moved J2 7.17 mm to (154.7, 40.5)
- moved J5 7.17 mm to (153.7, 41.0)
- moved J6 6.75 mm to (154.7, 41.6)
- moved P.2 6.73 mm to (160.3, 44.5)
- moved J3 6.68 mm to (155.7, 41.0)
- moved J7 6.41 mm to (155.7, 42.1)
- moved J4 6.25 mm to (156.8, 41.6)
- moved J8 6.15 mm to (156.8, 42.6)
- moved PH_Pitch2.54 5.32 mm to (165.2, 41.7), turned to 0 degrees
- moved P.3 5.22 mm to (161.0, 47.2)
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- renumbered R0603(0201) to R0603(0201)1, R1005(0402) to R1005(0402)1, R1608(0603) to R1608(0603)1, R2012(0805) to R2012(0805)1, R3216(1206) to R3216(1206)1, R3225(1210) to R3225(1210)1
Routing:
- net Net-(J4-Pad1): track 81.4 -> 60.3 mm
- net Net-(J1-Pad1): track 89.9 -> 68.9 mm
- net Net-(J2-Pad1): track 87.4 -> 66.8 mm
- net Net-(J3-Pad1): track 84.8 -> 64.3 mm
Other:
- board size 31 x 22.5 mm -> 23 x 18 mm
- board text added: "(0805)"
- board text added: "(1206)"
- board text added: "(1210)"
- board text added: ".5"
- board text added: ".5/.25"
- board text added: ".65"
- board text added: ".65/.3"
- board text added: ".8"
- board text added: ".8/.35"
- board text added: "1.0/.4"
- board text added: "18x22mm"
- board text added: "2.5/5/10/20mil"
- board text added: "R0603(0201)"
- board text added: "R1005(0402)"
- board text added: "R1608(0603)"
- board text added: "R2012"
- board text added: "R3216"
- board text added: "R3225"
- board text added: "w0.4/"
- board text removed: "0.25"
- board text removed: "0.3"
- board text removed: "0.35"
- board text removed: "0.4"
- board text removed: "0.5"
- board text removed: "0.5mm"
- board text removed: "0.65"
- board text removed: "0.65mm"
- board text removed: "0.8"
- board text removed: "0.8mm"
- board text removed: "1.0mm"
- board text removed: "10/20mil"
- board text removed: "2.5/5"
- board text removed: "22.5x31mm"
- board text removed: "by Shingo"
- board text removed: "w0.4"
