File: kicad/fiberPCB/test02.kicad_pcb (KiCad board)
At the start: 2 copper layers, 31 x 19 mm, 14 parts, among them J1 Barrel_Jack_Switch, U1 TC7WZ08FK

Commit message: add step2_drilll
Other:
- board text added: "19x31mm"

Commit message: add step2_drilll
Other:
- board size 31 x 19 mm -> 30 x 18 mm
- board text added: "18x30mm"
- board text removed: "19x31mm"

Commit message: update test02
Parts:
- J1: moved to B.Cu
- moved J1 10.0 mm to (143.0, 81.0), turned to 270 degrees
Routing:
- net VCC: track 55.6 -> 57.7 mm
- net GND: track 32.4 -> 33.5 mm

Commit message: update test02
Routing:
- net GND: track 33.5 -> 35.6 mm
Other:
- board size 30 x 18 mm -> 29 x 16.5 mm
- board text added: "16.5x29mm"
- board text removed: "18x30mm"
Changed lines of the file:
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@@
     (thickness 1.6)
     (drawings 16)
-    (tracks 84)
+    (tracks 86)
     (zones 0)
     (modules 14)
@@
     )
   )
-  (gr_text 18x30mm (at 142 66) (layer Dwgs.User)
+  (gr_text 16.5x29mm (at 142 66) (layer Dwgs.User)
     (effects (font (size 1 1) (thickness 0.15)))
   )
@@
     (effects (font (size 1 1) (thickness 0.25)))
   )
-  (gr_line (start 138 85) (end 138 67) (layer Edge.Cuts) (width 0.1))
-  (gr_line (start 168 85) (end 138 85) (layer Edge.Cuts) (width 0.1))
-  (gr_line (start 168 67) (end 168 85) (layer Edge.Cuts) (width 0.1))
-  (gr_line (start 138 67) (end 168 67) (layer Edge.Cuts) (width 0.1))
-  (gr_text "fiberPCB test02" (at 162.5 83.75) (layer F.Cu)
+  (gr_line (start 138 83.5) (end 138 67) (layer Edge.Cuts) (width 0.1))
+  (gr_line (start 167 83.5) (end 138 83.5) (layer Edge.Cuts) (width 0.1))
+  (gr_line (start 167 67) (end 167 83.5) (layer Edge.Cuts) (width 0.1))
+  (gr_line (start 138 67) (end 167 67) (layer Edge.Cuts) (width 0.1))
+  (gr_text "fiberPCB test02" (at 144 71.5) (layer F.Cu)
     (effects (font (size 0.8 0.8) (thickness 0.2)))
   )
@@
     (effects (font (size 1 1) (thickness 0.25)))
   )
-  (gr_text 2B (at 166.07244 81.48828) (layer F.Cu)
-    (effects (font (size 1 1) (thickness 0.25)))
-  )
-  (gr_text 2A (at 166.07244 78.82128) (layer F.Cu)
-    (effects (font (size 1 1) (thickness 0.25)))
-  )
-  (gr_text 1B (at 166.07244 71.70674) (layer F.Cu)
-    (effects (font (size 1 1) (thickness 0.25)))
-  )
-  (gr_text 1A (at 166.07244 69.04228) (layer F.Cu)
-    (effects (font (size 1 1) (thickness 0.25)))
+  (gr_text 2B (at 165.57244 81.48828) (layer F.Cu)
+    (effects (font (size 0.8 0.8) (thickness 0.2)))
+  )
+  (gr_text 2A (at 165.57244 78.82128) (layer F.Cu)
+    (effects (font (size 0.8 0.8) (thickness 0.2)))
+  )
+  (gr_text 1B (at 165.57244 71.70674) (layer F.Cu)
+    (effects (font (size 0.8 0.8) (thickness 0.2)))
+  )
+  (gr_text 1A (at 165.57244 69.04228) (layer F.Cu)
+    (effects (font (size 0.8 0.8) (thickness 0.2)))
   )
   (gr_text 2Y (at 150.75 75.25) (layer F.Cu)
@@
   (segment (start 157.65508 80.09492) (end 157.65508 79.62156) (width 0.25) (layer F.Cu) (net 4))
   (segment (start 157.65508 81.36128) (end 157.65508 80.09492) (width 0.25) (layer F.Cu) (net 4))
-  (segment (start 148.259534 69.740466) (end 157.086434 69.740466) (width 0.25) (layer F.Cu) (net 4))
-  (segment (start 157.086434 69.740466) (end 157.65508 69.17182) (width 0.25) (layer F.Cu) (net 4))
-  (segment (start 143 75) (end 148.259534 69.740466) (width 0.25) (layer F.Cu) (net 4))
+  (segment (start 151.382246 69.17182) (end 157.65508 69.17182) (width 0.25) (layer F.Cu) (net 4))
+  (segment (start 150 74) (end 150 70.554066) (width 0.25) (layer F.Cu) (net 4))
+  (segment (start 149 75) (end 150 74) (width 0.25) (layer F.Cu) (net 4))
+  (segment (start 150 70.554066) (end 151.382246 69.17182) (width 0.25) (layer F.Cu) (net 4))
+  (segment (start 143 75) (end 149 75) (width 0.25) (layer F.Cu) (net 4))
   (segment (start 161.91508 78.82128) (end 159.50508 78.82128) (width 0.25) (layer F.Cu) (net 5))
   (segment (start 162.31508 78.42128) (end 161.91508 78.82128) (width 0.25) (layer F.Cu) (net 5))
